File: power.kicad_sch (KiCad schematic)
At the start: 0 parts

Commit message: add buck and power switch
Parts:
- added C1: 10uF, symbol Device:C
- added C2: 4.7uF, symbol Device:C
- added C3: 100nF, symbol Device:C
- added D1, D2: D_Schottky, symbol Device:D_Schottky
- added J4: Conn_Coaxial_Small, symbol Connector:Conn_Coaxial_Small
- added J5: batt, symbol Connector_Generic:Conn_01x02
- added L1: 2.2uH, symbol Device:L
- added Q1, Q2: PMOS, symbol Simulation_SPICE:PMOS
- added R10: 150K, symbol Device:R
- added R11: 100k, symbol Device:R
- added R9: 680k, symbol Device:R
- added SW41: SW_SPDT, symbol Switch:SW_SPDT
- added U4: TLV62569DBV, Package_TO_SOT_SMD:SOT-23-5, symbol Regulator_Switching:TLV62569DBV
Connections:
- new net: C3.1, J5.2 (Pin_2), Q1.1 (D)
- new net: Q1.3 (S), Q2.3 (S), SW41.3 (C)
- new net: R10.1, R9.2, U4.5 (FB)
- new net: J4.2 (Ext), L1.1, U4.3 (SW)
- new net: Q2.2 (G), R11.2
- new net: R11.1, SW41.2 (B)
- new net +3.3V: C1.1, L1.2, R9.1
- new net +BATT: D1.2 (A), Q2.1 (D)
- new net GND: C1.2, C2.2, C3.2, J4.1 (In), J5.1 (Pin_1), Q1.2 (G), R10.2, SW41.1 (A), U4.2 (GND)
- new net VBUS: D2.2 (A)
- new net VDD: C2.1, D1.1 (K), D2.1 (K), U4.1 (EN), U4.4 (VIN)
Other:
- note added: "https://wmsc.lcsc.com/wmsc/upload/file/pdf/v2/lcsc/1809251629_Texas-Instruments-TLV62569DBVR_C141836.pdf"
